File: gk/interface.kicad_sch (KiCad schematic)
At the start: 60 parts, among them U9 LSM6DSL

Commit message: Update pcb
Parts:
- added J11: Conn_01x02, Connector_JST:JST_XH_S2B-XH-A_1x02_P2.50mm_Horizontal, symbol Connector_Generic:Conn_01x02
- added R57: 10k, Resistor_SMD:R_0603_1608Metric, symbol Device:R
- added SW3: RotaryEncoder_Switch, Rotary_Encoder:RotaryEncoder_Alps_EC11E-Switch_Vertical_H20mm, symbol Device:RotaryEncoder_Switch
Connections:
- net GND: now also R57.2, SW3.C, SW3.S2
- net VCC: now also J11.1 (Pin_1)
- net at R36.2, R37.1, SW_U1.2: now also SW3.A
- net at R38.2, R39.1, SW_D1.2: now also SW3.B
- net at R40.2, R41.1, SW_L1.2: now also SW3.S1
- net LSM6DSL_INT2: no longer names the net of U9.9 (INT2)
- new net NTC_MCU: J11.2 (Pin_2), R57.1
- no-connect marks 9 -> 10
