File: gk-pcbv2/gk-pcbv2/audio.kicad_sch (KiCad schematic)
At the start: 33 parts, among them J5 AudioJack3_SwitchTR, J6 Conn_01x02, U12 PAM8302AAS, U14 TPA6110A2DGN, U7 PCM1753DBQ

Commit message: more v2 pcb changes
Connections:
- net VCC: no longer C80.1, C81.1, U12.6 (VDD)
- net VDDA: now also C80.1, C81.1, U12.6 (VDD)
Changed lines of the file:
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@@
     )
   )
-  (symbol (lib_id "power:VCC") (at 69.85 123.19 0) (unit 1)
+  (symbol (lib_id "power:VDDA") (at 69.85 123.19 0) (unit 1)
     (in_bom yes) (on_board yes) (dnp no) (fields_autoplaced)
-    (property "Reference" "#PWR076" (at 69.85 127 0)
+    (property "Reference" "#PWR05" (at 69.85 127 0)
       (effects (font (size 1.27 1.27)) hide)
     )
-    (property "Value" "VCC" (at 69.85 119.38 0)
+    (property "Value" "VDDA" (at 69.85 118.11 0)
       (effects (font (size 1.27 1.27)))
     )
@@
       (project "gk-pcbv2"
         (path "/08730ac6-6084-459f-bdf1-86b322355ede/10bf96f0-351a-4550-b62a-cc824dccdbb6"
-          (reference "#PWR076") (unit 1)
+          (reference "#PWR05") (unit 1)
         )
       )
