File: gk-pcbv2/gk-pcbv2/gk-pcbv2.kicad_sch (KiCad schematic)
At the start: 73 parts, among them J1 USB_C_Receptacle_USB2.0, J10 Barrel_Jack_Switch, J2 Conn_01x02, J8 Conn_ARM_JTAG_SWD_10, U1 WE-TVS-82400102, U10 MAX17048, U13 LTC3536xMSE, U15 MAX40203AUK, U16 MAX40203AUK, U2 MCP73831-2-OT, U3 AP62300WU

Commit message: more v2 pcb changes
Parts:
- added J12: Conn_01x02, Connector_PinHeader_2.54mm:PinHeader_1x02_P2.54mm_Vertical, symbol Connector_Generic:Conn_01x02
- added R79: Rsense, Resistor_SMD:R_2512_6332Metric, symbol Device:R
Connections:
- net VCC: now also J12.1 (Pin_1), R79.1; no longer C85.1, C87.1, R74.1, U13.7 (VOUT)
- new net: C85.1, C87.1, J12.2 (Pin_2), R74.1, R79.2, U13.7 (VOUT)
Changed lines of the file:
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@@
   (junction (at 137.16 55.88) (diameter 0) (color 0 0 0 0)
   )
-  (junction (at 267.97 45.72) (diameter 0) (color 0 0 0 0)
-  )
   (junction (at 149.86 105.41) (diameter 0) (color 0 0 0 0)
   )
@@
   (junction (at 220.98 72.39) (diameter 0) (color 0 0 0 0)
   )
+  (junction (at 267.97 44.45) (diameter 0) (color 0 0 0 0)
+  )
   (junction (at 50.8 118.11) (diameter 0) (color 0 0 0 0)
   )
@@
   (junction (at 214.63 139.7) (diameter 0) (color 0 0 0 0)
   )
+  (junction (at 267.97 45.72) (diameter 0) (color 0 0 0 0)
+  )
   (junction (at 168.91 45.72) (diameter 0) (color 0 0 0 0)
   )
@@
   (junction (at 146.05 55.88) (diameter 0) (color 0 0 0 0)
   )
+  (junction (at 267.97 36.83) (diameter 0) (color 0 0 0 0)
+  )
   (junction (at 106.68 88.9) (diameter 0) (color 0 0 0 0)
   )
@@
     (stroke (width 0) (type default))
   )
+  (wire (pts (xy 265.43 41.91) (xy 262.89 41.91))
+    (stroke (width 0) (type default))
+  )
   (wire (pts (xy 81.28 21.59) (xy 81.28 24.13))
     (stroke (width 0) (type default))
@@
     (stroke (width 0) (type default))
   )
-  (wire (pts (xy 267.97 45.72) (xy 271.78 45.72))
-    (stroke (width 0) (type default))
-  )
   (wire (pts (xy 109.22 88.9) (xy 106.68 88.9))
     (stroke (width 0) (type default))
@@
     (stroke (width 0) (type default))
   )
+  (wire (pts (xy 267.97 44.45) (xy 265.43 44.45))
+    (stroke (width 0) (type default))
+  )
   (wire (pts (xy 86.36 60.96) (xy 86.36 62.23))
     (stroke (width 0) (type default))
@@
     (stroke (width 0) (type default))
   )
+  (wire (pts (xy 267.97 44.45) (xy 267.97 45.72))
+    (stroke (width 0) (type default))
+  )
+  (wire (pts (xy 267.97 35.56) (xy 267.97 36.83))
+    (stroke (width 0) (type default))
+  )
   (wire (pts (xy 113.03 115.57) (xy 135.89 115.57))
     (stroke (width 0) (type default))
@@
     (stroke (width 0) (type default))
   )
+  (wire (pts (xy 265.43 39.37) (xy 265.43 36.83))
+    (stroke (width 0) (type default))
+  )
   (wire (pts (xy 74.93 132.08) (xy 87.63 132.08))
     (stroke (width 0) (type default))
@@
     (stroke (width 0) (type default))
   )
+  (wire (pts (xy 265.43 36.83) (xy 267.97 36.83))
+    (stroke (width 0) (type default))
+  )
   (wire (pts (xy 129.54 27.94) (xy 129.54 29.21))
     (stroke (width 0) (type default))
@@
     (stroke (width 0) (type default))
   )
+  (wire (pts (xy 267.97 45.72) (xy 271.78 45.72))
+    (stroke (width 0) (type default))
+  )
+  (wire (pts (xy 262.89 39.37) (xy 265.43 39.37))
+    (stroke (width 0) (type default))
+  )
   (wire (pts (xy 50.8 110.49) (xy 59.69 110.49))
     (stroke (width 0) (type default))
@@
     (stroke (width 0) (type default))
   )
+  (wire (pts (xy 265.43 44.45) (xy 265.43 41.91))
+    (stroke (width 0) (type default))
+  )
   (wire (pts (xy 62.23 132.08) (xy 74.93 132.08))
     (stroke (width 0) (type default))
@@
     )
   )
+  (symbol (lib_id "Connector_Generic:Conn_01x02") (at 257.81 39.37 0) (mirror y) (unit 1)
+    (in_bom yes) (on_board yes) (dnp no) (fields_autoplaced)
+    (property "Reference" "J12" (at 257.81 33.02 0)
+      (effects (font (size 1.27 1.27)))
+    )
+    (property "Value" "Conn_01x02" (at 257.81 35.56 0)
+      (effects (font (size 1.27 1.27)))
+    )
+    (property "Footprint" "Connector_PinHeader_2.54mm:PinHeader_1x02_P2.54mm_Vertical" (at 257.81 39.37 0)
+      (effects (font (size 1.27 1.27)) hide)
+    )
+    (property "Datasheet" "~" (at 257.81 39.37 0)
+      (effects (font (size 1.27 1.27)) hide)
+    )
+    (pin "1")
+    (pin "2")
+    (instances
+      (project "gk-pcbv2"
+        (path "/08730ac6-6084-459f-bdf1-86b322355ede"
+          (reference "J12") (unit 1)
+        )
+      )
+    )
+  )
   (symbol (lib_id "power:VCC") (at 36.83 132.08 0) (unit 1)
     (in_bom yes) (on_board yes) (dnp no) (fields_autoplaced)
@@
     )
   )
-  (symbol (lib_id "power:VCC") (at 267.97 45.72 0) (unit 1)
+  (symbol (lib_id "power:VCC") (at 267.97 35.56 0) (unit 1)
     (in_bom yes) (on_board yes) (dnp no) (fields_autoplaced)
-    (property "Reference" "#PWR02" (at 267.97 49.53 0)
+    (property "Reference" "#PWR02" (at 267.97 39.37 0)
       (effects (font (size 1.27 1.27)) hide)
     )
-    (property "Value" "VCC" (at 267.97 41.91 0)
+    (property "Value" "VCC" (at 267.97 31.75 0)
       (effects (font (size 1.27 1.27)))
     )
-    (property "Footprint" "" (at 267.97 45.72 0)
+    (property "Footprint" "" (at 267.97 35.56 0)
       (effects (font (size 1.27 1.27)) hide)
     )
-    (property "Datasheet" "" (at 267.97 45.72 0)
+    (property "Datasheet" "" (at 267.97 35.56 0)
       (effects (font (size 1.27 1.27)) hide)
     )
@@
         )
       )
+    )
+  )
+  (symbol (lib_id "Device:R") (at 267.97 40.64 0) (unit 1)
+    (in_bom yes) (on_board yes) (dnp no) (fields_autoplaced)
+    (property "Reference" "R79" (at 270.51 39.37 0)
+      (effects (font (size 1.27 1.27)) (justify left))
+    )
+    (property "Value" "Rsense" (at 270.51 41.91 0)
+      (effects (font (size 1.27 1.27)) (justify left))
+    )
+    (property "Footprint" "Resistor_SMD:R_2512_6332Metric" (at 266.192 40.64 90)
+      (effects (font (size 1.27 1.27)) hide)
+    )
+    (property "Datasheet" "~" (at 267.97 40.64 0)
+      (effects (font (size 1.27 1.27)) hide)
+    )
+    (pin "1")
+    (pin "2")
+    (instances
+      (project "gk-pcbv2"
+        (path "/08730ac6-6084-459f-bdf1-86b322355ede"
+          (reference "R79") (unit 1)
+        )
+      )

Commit message: more pcb changes
Parts:
- added TP1, TP2, TP3, TP4, TP5, TP6, TP7, TP8: TestPoint, Connector_PinHeader_2.54mm:PinHeader_1x01_P2.54mm_Vertical, symbol Connector:TestPoint
- R79: value Rsense -> 0R / 1m-5m
Connections:
- net GND: now also TP6.1, TP7.1, TP8.1
- net USB_VBUS: now also TP4.1
- net VCC: now also TP1.1
- net VREGIN: now also TP2.1
- net VLITH: now reaches C2.1, C79.1, J2.1 (Pin_1), R54.1, U10.2 (CELL), U10.3 (VDD), U15.1 (VDD), U15.3 (EN), U16.1 (VDD), U16.3 (EN), U2.3 (V_{BAT})
- net VLITH: now also TP3.1
- new net VDDA: TP5.1
