File: gk-pcbv3/gk-pcbv3/gk-pcbv3.kicad_sch (KiCad schematic)
At the start: 38 parts, among them J1 USB_C_Receptacle_USB2.0, J14 USB_A, J2 Conn_01x02, J7 Conn_01x02, J8 Conn_ARM_JTAG_SWD_10, U1 WE-TVS-82400102, U10 MAX17048, U21 BQ24075RGT, U23 WE-TVS-82400102, U24 TPS2051CDBV

Commit message: new gerbers
Parts:
- added R11: NC/10k, Resistor_SMD:R_0603_1608Metric, symbol Device:R
- J7: footprint Connector_JST:JST_XH_S2B-XH-A_1x02_P2.50mm_Horizontal -> Connector_JST:JST_XH_B2B-XH-A_1x02_P2.50mm_Vertical
- JP4: footprint (none) -> Jumper:SolderJumper-2_P1.3mm_Open_Pad1.0x1.5mm
- U21: value BQ24075RGT -> BQ24075RGT (_not_ BQ24075*T*RGT)
Connections:
- net GND: now also J2.1 (Pin_1), R11.1; no longer J2.2 (Pin_2)
- net VLITH: now also J2.2 (Pin_2); no longer J2.1 (Pin_1)
- net at J7.1 (Pin_1), U21.1 (TS): now also R11.2
Other:
- moved on the sheet: J2, J7
Changed lines of the file:
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@@
 	)
 	(junction
-		(at 177.8 72.39)
+		(at 180.34 53.34)
 		(diameter 0)
 		(color 0 0 0 0)
@@
 	)
 	(junction
+		(at 189.23 72.39)
+		(diameter 0)
+		(color 0 0 0 0)
+	)
+	(junction
+		(at 180.34 72.39)
+		(diameter 0)
+		(color 0 0 0 0)
+	)
+	(junction
+		(at 203.2 55.88)
+		(diameter 0)
+		(color 0 0 0 0)
+	)
+	(junction
 		(at 60.96 72.39)
 		(diameter 0)
@@
 	)
 	(junction
-		(at 203.2 55.88)
-		(diameter 0)
-		(color 0 0 0 0)
-	)
-	(junction
 		(at 19.05 102.87)
 		(diameter 0)
@@
 	(wire
 		(pts
-			(xy 203.2 55.88) (xy 203.2 59.69)
+			(xy 203.2 55.88) (xy 203.2 60.96)
 		)
 		(stroke
@@
 	(wire
 		(pts
-			(xy 177.8 55.88) (xy 177.8 72.39)
-		)
-		(stroke
-			(width 0)
-			(type default)
-		)
-	)
-	(wire
-		(pts
 			(xy 129.54 59.69) (xy 107.95 59.69)
 		)
@@
 	(wire
 		(pts
+			(xy 203.2 55.88) (xy 238.76 55.88)
+		)
+		(stroke
+			(width 0)
+			(type default)
+		)
+	)
+	(wire
+		(pts
 			(xy 44.45 130.81) (xy 44.45 129.54)
 		)
@@
 	(wire
 		(pts
+			(xy 180.34 72.39) (xy 189.23 72.39)
+		)
+		(stroke
+			(width 0)
+			(type default)
+		)
+	)
+	(wire
+		(pts
 			(xy 44.45 107.95) (xy 52.07 107.95)
 		)
@@
 	(wire
 		(pts
-			(xy 238.76 55.88) (xy 203.2 55.88)
+			(xy 193.04 55.88) (xy 203.2 55.88)
 		)
 		(stroke
@@
 	(wire
 		(pts
-			(xy 177.8 72.39) (xy 193.04 72.39)
+			(xy 142.24 72.39) (xy 180.34 72.39)
 		)
 		(stroke
@@
 	(wire
 		(pts
+			(xy 180.34 63.5) (xy 180.34 72.39)
+		)
+		(stroke
+			(width 0)
+			(type default)
+		)
+	)
+	(wire
+		(pts
+			(xy 182.88 57.15) (xy 189.23 57.15)
+		)
+		(stroke
+			(width 0)
+			(type default)
+		)
+	)
+	(wire
+		(pts
 			(xy 195.58 121.92) (xy 194.31 121.92)
 		)
@@
 	(wire
 		(pts
-			(xy 189.23 55.88) (xy 193.04 55.88)
+			(xy 189.23 57.15) (xy 189.23 72.39)
 		)
 		(stroke
@@
 	(wire
 		(pts
-			(xy 203.2 72.39) (xy 203.2 62.23)
+			(xy 189.23 55.88) (xy 193.04 55.88)
 		)
 		(stroke
@@
 	(wire
 		(pts
-			(xy 177.8 53.34) (xy 158.75 53.34)
+			(xy 158.75 53.34) (xy 180.34 53.34)
 		)
 		(stroke
@@
 	(wire
 		(pts
-			(xy 142.24 72.39) (xy 177.8 72.39)
+			(xy 154.94 49.53) (xy 173.99 49.53)
 		)
 		(stroke
@@
 	(wire
 		(pts
-			(xy 154.94 49.53) (xy 173.99 49.53)
+			(xy 58.42 33.02) (xy 58.42 50.8)
 		)
 		(stroke
@@
 	(wire
 		(pts
-			(xy 58.42 33.02) (xy 58.42 50.8)
+			(xy 180.34 53.34) (xy 180.34 55.88)
 		)
 		(stroke
@@
 	(wire
 		(pts
-			(xy 107.95 59.69) (xy 107.95 64.77)
+			(xy 180.34 53.34) (xy 180.34 50.8)
 		)
 		(stroke
@@
 	(wire
 		(pts
-			(xy 163.83 41.91) (xy 154.94 41.91)
+			(xy 107.95 59.69) (xy 107.95 64.77)
 		)
 		(stroke
@@
 	(wire
 		(pts
-			(xy 228.6 68.58) (xy 238.76 68.58)
+			(xy 163.83 41.91) (xy 154.94 41.91)
 		)
 		(stroke
@@
 	(wire
 		(pts
-			(xy 78.74 53.34) (xy 83.82 53.34)
+			(xy 228.6 68.58) (xy 238.76 68.58)
 		)
 		(stroke
@@
 	(wire
 		(pts
-			(xy 193.04 55.88) (xy 203.2 55.88)
+			(xy 78.74 53.34) (xy 83.82 53.34)
 		)
 		(stroke
@@
 	(wire
 		(pts
+			(xy 189.23 72.39) (xy 193.04 72.39)
+		)
+		(stroke
+			(width 0)
+			(type default)
+		)
+	)
+	(wire
+		(pts
 			(xy 241.3 63.5) (xy 238.76 63.5)
 		)
@@
 	(wire
 		(pts
+			(xy 182.88 50.8) (xy 182.88 57.15)
+		)
+		(stroke
+			(width 0)
+			(type default)
+		)
+	)
+	(wire
+		(pts
 			(xy 252.73 76.2) (xy 252.73 77.47)
 		)
@@
 	(wire
 		(pts
+			(xy 203.2 63.5) (xy 203.2 72.39)
+		)
+		(stroke
+			(width 0)
+			(type default)
+		)
+	)
+	(wire
+		(pts
 			(xy 254 74.93) (xy 254 76.2)
 		)
@@
 	(symbol
 		(lib_id "Connector_Generic:Conn_01x02")
-		(at 208.28 59.69 0)
+		(at 208.28 63.5 0)
+		(mirror x)
 		(unit 1)
 		(exclude_from_sim no)
@@
 		(on_board yes)
 		(dnp no)
-		(fields_autoplaced yes)
 		(property "Reference" "J2"
-			(at 210.82 60.325 0)
+			(at 210.82 62.865 0)
 			(effects
 				(font
@@
 		)
 		(property "Value" "Conn_01x02"
-			(at 210.82 62.865 0)
+			(at 210.82 60.325 0)
 			(effects
 				(font
@@
 		)
 		(property "Footprint" "Connector_JST:JST_PH_B2B-PH-K_1x02_P2.00mm_Vertical"
-			(at 208.28 59.69 0)
+			(at 208.28 63.5 0)
 			(effects
 				(font
@@
 		)
 		(property "Datasheet" "~"
-			(at 208.28 59.69 0)
+			(at 208.28 63.5 0)
 			(effects
 				(font
@@
 		)
 		(property "Description" ""
-			(at 208.28 59.69 0)
+			(at 208.28 63.5 0)
 			(effects
 				(font
@@
 			)
 		)
-		(property "Value" "BQ24075RGT"
+		(property "Value" "BQ24075RGT (_not_ BQ24075*T*RGT)"
 			(at 144.4341 36.83 0)
 			(effects
@@
 	)
 	(symbol
+		(lib_id "Device:R")
+		(at 180.34 59.69 180)
+		(unit 1)
+		(exclude_from_sim no)
+		(in_bom yes)
+		(on_board yes)
+		(dnp no)
+		(fields_autoplaced yes)
+		(property "Reference" "R11"
+			(at 182.88 58.4199 0)
+			(effects
+				(font
+					(size 1.27 1.27)
+				)
+				(justify right)
+			)
+		)
+		(property "Value" "NC/10k"
+			(at 182.88 60.9599 0)
+			(effects
+				(font
+					(size 1.27 1.27)
+				)
+				(justify right)
+			)
+		)
+		(property "Footprint" "Resistor_SMD:R_0603_1608Metric"
+			(at 182.118 59.69 90)
+			(effects
+				(font
+					(size 1.27 1.27)
+				)
+				(hide yes)
+			)
+		)
+		(property "Datasheet" "~"
+			(at 180.34 59.69 0)
+			(effects
+				(font
+					(size 1.27 1.27)
+				)
+				(hide yes)
+			)
+		)
+		(property "Description" ""
+			(at 180.34 59.69 0)
+			(effects
+				(font
+					(size 1.27 1.27)
+				)
+				(hide yes)
+			)
+		)
+		(pin "1"
+		)
+		(pin "2"
+		)
+		(instances
+			(project "gk-pcbv3"
+				(path "/08730ac6-6084-459f-bdf1-86b322355ede"
+					(reference "R11")
+					(unit 1)
+				)
+			)
+		)
+	)
+	(symbol
 		(lib_id "Power_Protection:WE-TVS-82400102")
 		(at 59.69 132.08 0)
@@
 	(symbol
 		(lib_id "Connector_Generic:Conn_01x02")
-		(at 182.88 53.34 0)
+		(at 180.34 45.72 90)
 		(unit 1)
 		(exclude_from_sim no)
@@
 		(fields_autoplaced yes)
 		(property "Reference" "J7"
-			(at 182.88 48.26 0)
+			(at 185.42 44.4499 90)
 			(effects
 				(font
 					(size 1.27 1.27)
 				)
+				(justify right)
 			)
 		)
 		(property "Value" "Conn_01x02"
-			(at 182.88 50.8 0)
+			(at 185.42 46.9899 90)
 			(effects
 				(font
 					(size 1.27 1.27)
 				)
+				(justify right)
 			)
 		)
-		(property "Footprint" "Connector_JST:JST_XH_S2B-XH-A_1x02_P2.50mm_Horizontal"
-			(at 182.88 53.34 0)
+		(property "Footprint" "Connector_JST:JST_XH_B2B-XH-A_1x02_P2.50mm_Vertical"
+			(at 180.34 45.72 0)
 			(effects
 				(font
@@
 		)
 		(property "Datasheet" "~"
-			(at 182.88 53.34 0)
+			(at 180.34 45.72 0)
 			(effects
 				(font
@@
 		)
 		(property "Description" ""
-			(at 182.88 53.34 0)
+			(at 180.34 45.72 0)
 			(effects
 				(font
@@
 			)
 		)
-		(property "Footprint" ""
+		(property "Footprint" "Jumper:SolderJumper-2_P1.3mm_Open_Pad1.0x1.5mm"
 			(at 101.6 55.88 0)
 			(effects
