File: gk-pcbv4/pmic/pmic.kicad_pcb (KiCad board)
At the start: 4 copper layers, 25.4 x 25.4 mm, 50 parts, among them U1 STPMIC25BPQR

Commit message: pcb order 20251115
Parts:
- added D1: LED, LED_SMD:LED_0603_1608Metric, F.Cu at (125.0, 60.9)
- added R1: 1k, Resistor_SMD:R_0603_1608Metric, F.Cu at (122.0, 59.8)
Routing:
- net VOUT4: track 34.5 -> 52.2 mm, vias 2 -> 3
- net VIN: track 49.4 -> 57.7 mm
- net GND: track 58.4 -> 63.2 mm, vias 73 -> 72
- net Net-(D1-K): track 0.00 -> 2.15 mm
- net Net-(U1-VLX6): track 7.21 -> 7.78 mm
