File: gk-pcbv4/pmic/pmic.kicad_sch (KiCad schematic)
At the start: 50 parts, among them U1 STPMIC25BPQR

Commit message: pcb order 20251115
Parts:
- added D1: LED, LED_SMD:LED_0603_1608Metric, symbol Device:LED
- added R1: 1k, Resistor_SMD:R_0603_1608Metric, symbol Device:R
Connections:
- net GND: now also R1.2
- net VOUT4: now also D1.2 (A)
- new net: D1.1 (K), R1.1
