File: gk-pcbv4/oled_pcb/gk_oled_pcb/gk_oled_pcb.kicad_sch (KiCad schematic)
At the start: 48 parts, among them J2 Conn_01x01, J3 Conn_01x01, J4 Conn_01x06, J5 Conn_01x01, U1 TCA9546APW

Commit message: begin work on adding oled board to gk
Parts:
- JP1, JP2, JP3, JP4: footprint oled_lib:OLED_0_5inch_14pin -> oled_lib:FPC_0.62mm_14pin
Changed lines of the file:
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@@
 			)
 		)
-		(property "Footprint" "oled_lib:OLED_0_5inch_14pin"
+		(property "Footprint" "oled_lib:FPC_0.62mm_14pin"
 			(at 132.08 25.4 0)
 			(hide yes)
@@
 			)
 		)
-		(property "Footprint" "oled_lib:OLED_0_5inch_14pin"
+		(property "Footprint" "oled_lib:FPC_0.62mm_14pin"
 			(at 30.48 25.4 0)
 			(hide yes)
@@
 			)
 		)
-		(property "Footprint" "oled_lib:OLED_0_5inch_14pin"
+		(property "Footprint" "oled_lib:FPC_0.62mm_14pin"
 			(at 81.28 25.4 0)
 			(hide yes)
@@
 			)
 		)
-		(property "Footprint" "oled_lib:OLED_0_5inch_14pin"
+		(property "Footprint" "oled_lib:FPC_0.62mm_14pin"
 			(at 182.88 25.4 0)
 			(hide yes)
