File: gk-pcbv4/gk-controls/gk-controls.kicad_sch (KiCad schematic)
At the start: 41 parts, among them J1 Conn_01x20, J10 Conn_01x01, J7 Conn_01x06, J8 Conn_01x01, J9 Conn_01x01, U1 PCAL6416APW, U2 ULN2003A

Commit message: update controls layout triggers now are analog new ADC on control board Move bumper buttons to trigger daughterboard and put in more ergonomical position
Parts:
- added C25, C26, C27: 1u, Capacitor_SMD:C_0603_1608Metric, symbol Device:C
- added H5, H7: MountingHole, MountingHole:MountingHole_2.7mm_M2.5, symbol Mechanical:MountingHole
- added J11: Conn_01x06, Connector_FFC-FPC:TE_0-1734839-6_1x06-1MP_P0.5mm_Horizontal, symbol Connector_Generic:Conn_01x06
- added R50, R51, R52, R53: NC, Resistor_SMD:R_0603_1608Metric, symbol Device:R
- added U5: (no value), Package_DFN_QFN:WQFN-16-1EP_3x3mm_P0.5mm_EP1.6x1.6mm_ThermalVias, symbol ads7138:ADS7138
- R11, R47, R48, R49: value 10k -> 10k/0R
Connections:
- net GND: now also C25.2, C26.2, C27.2, J11.1 (Pin_1), U5.17, U5.5 (IO6), U5.6 (IO7), U5.9 (GND)
- net I2C1_SCL: now also U5.13 (SCL)
- net I2C1_SDA: now also U5.14 (SDA)
- net JOY_A_X: now also R51.1, U5.1 (IO2)
- net JOY_A_Y: now also R50.1, U5.2 (IO3)
- net JOY_B_X: now also R52.1, U5.3 (IO4)
- net JOY_B_Y: now also R53.1, U5.4 (IO5)
- net VDDA: now also C26.1, J11.6 (Pin_6), U5.7 (AVDD)
- net VDDIO: now also C27.1, U5.10 (DVDD)
- net BTN_MCU_LT renamed BTN_MCU_LB
- net BTN_MCU_RT renamed BTN_MCU_RB
- net JOY_A_X_MCU: no longer names the net of J1.3 (Pin_3)
- net JOY_A_X_MCU: now also R51.2
- net JOY_A_Y_MCU: no longer names the net of J1.5 (Pin_5)
- net JOY_A_Y_MCU: now also R50.2
- net JOY_B_X_MCU: no longer names the net of J1.7 (Pin_7)
- net JOY_B_X_MCU: now also R52.2
- net JOY_B_Y_MCU: no longer names the net of J1.9 (Pin_9)
- net JOY_B_Y_MCU: now also R53.2
- new net: C25.1, U5.11 (ADDR), U5.8 (DECAP)
- new net BTN_LB: J11.5 (Pin_5)
- new net BTN_RB: J11.4 (Pin_4)
- new net LT_ANA: J11.3 (Pin_3), U5.15 (IO0)
- new net RT_ANA: J11.2 (Pin_2), U5.16 (IO1)
- no-connect marks 4 -> 5
Other:
- note added: "Connection to button OLED board and mount holes"
- note added: "Connection to trigger board Inverted wrt trigger board pins as on opposite side of board"
- note added: "Extra ADC. Can also use IO pins as GPIOs. Programmed for I2C addr 0x17"
- note added: "Menu button LED driver"
- note added: "Option to use CM33 ADC or ADS7138 here"
- moved on the sheet: BT1, C10, C9, D1, D2, H1, H2, H3, H4, H6, H8, H9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
